Commit message: add kdl checker

File: cw3_stack/iiwa_description/urdf/iiwa14.xacro (robot description, xacro)
@@ -12,6 +12,6 @@
   <xacro:property name="safety_controller_k_vel" value="2" />
   <xacro:property name="joint_damping" value="0.5" />
-  <xacro:property name="max_effort" value="300"/>
-  <xacro:property name="max_velocity" value="100"/>
+  <xacro:property name="max_effort" value="100"/>
+  <xacro:property name="max_velocity" value="20"/>
   <xacro:macro name="iiwa14" params="parent hardware_interface robot_name *origin">
     <!--joint between {parent} and link_0-->

Commit message: Fix robot urdf

File: cw3_stack/iiwa_description/urdf/iiwa14.xacro (robot description, xacro)
@@ -12,6 +12,6 @@
   <xacro:property name="safety_controller_k_vel" value="2" />
   <xacro:property name="joint_damping" value="0.5" />
-  <xacro:property name="max_effort" value="100"/>
-  <xacro:property name="max_velocity" value="20"/>
+  <xacro:property name="max_effort" value="300"/>
+  <xacro:property name="max_velocity" value="100"/>
   <xacro:macro name="iiwa14" params="parent hardware_interface robot_name *origin">
     <!--joint between {parent} and link_0-->
